Commit message: Modificado urdf para agregar todos los sensores

File: rover_description/src/description/rover.urdf (robot description, URDF)
Before this commit: robot sam_bot, 3 links, 2 joints
Links:
- added link camera_left; visual box size=0.01 0.01 0.01
- added link camera_right; visual box size=0.01 0.01 0.01
- added link deph; visual box size=0.01 0.01 0.01
- added link gps; visual box size=0.01 0.01 0.01
- added link imu; visual box size=0.01 0.01 0.01
- added link lidar; visual cylinder length=0.05 radius=0.05
Joints:
- added joint camera_left_joint: type fixed, parent base_link, child camera_left, origin xyz=0.405 0.03 ${height+0.095} rpy=0 0 -1.5708
- added joint camera_right_joint: type fixed, parent base_link, child camera_right, origin xyz=0.405 -0.03 ${height+0.095} rpy=0 0 -1.5708
- added joint deph_joint: type fixed, parent base_link, child deph, origin xyz=0.405 0.0 ${height+0.095} rpy=0 0 -1.5708
- added joint gps_joint: type fixed, parent base_link, child gps, origin xyz=-0.1 0.0 ${height+0.105} rpy=0 0 -1.5708
- added joint imu_joint: type fixed, parent base_link, child imu, origin xyz=0.0 0.0 ${height+0.105} rpy=0 0 -1.5708
- added joint lidar_joint: type fixed, parent base_link, child lidar, origin xyz=0.22 0.0 ${height+0.125} rpy=0 0 -1.5708
- joint camera_joint: origin xyz=0.39 0.0 0.61 rpy=0 0 -1.5708 -> xyz=0.39 0.0 ${height+0.11} rpy=0 0 -1.5708

Commit message: Añadidas algunas caracteristicas de los sensores, falta el motion blur del range finder y todo de las camaras

File: rover_description/src/description/rover.urdf (robot description, URDF)
Before this commit: robot sam_bot, 9 links, 8 joints
Joints:
- joint camera_left_joint: origin xyz=0.405 0.03 ${height+0.095} rpy=0 0 -1.5708 -> xyz=0.405 0.06 ${height+0.095} rpy=0 0 -1.5708
- joint camera_right_joint: origin xyz=0.405 -0.03 ${height+0.095} rpy=0 0 -1.5708 -> xyz=0.405 -0.06 ${height+0.095} rpy=0 0 -1.5708

Commit message: Arreglado publicaciones de sensores según marcos de referencia

File: rover_description/src/description/rover.urdf (robot description, URDF)
Before this commit: robot sam_bot, 9 links, 8 joints
Joints:
- joint camera_joint: origin xyz=0.39 0.0 ${height+0.11} rpy=0 0 -1.5708 -> xyz=0.39 0.0 ${height+0.11} rpy=0 0 0
- joint camera_left_joint: origin xyz=0.405 0.06 ${height+0.095} rpy=0 0 -1.5708 -> xyz=0.405 0.06 ${height+0.095} rpy=0 0 0
- joint camera_right_joint: origin xyz=0.405 -0.06 ${height+0.095} rpy=0 0 -1.5708 -> xyz=0.405 -0.06 ${height+0.095} rpy=0 0 0
- joint deph_joint: origin xyz=0.405 0.0 ${height+0.095} rpy=0 0 -1.5708 -> xyz=0.405 0.0 ${height+0.095} rpy=0 0 0
- joint gps_joint: origin xyz=-0.1 0.0 ${height+0.105} rpy=0 0 -1.5708 -> xyz=-0.1 0.0 ${height+0.105} rpy=0 0 0
- joint imu_joint: origin xyz=0.0 0.0 ${height+0.105} rpy=0 0 -1.5708 -> xyz=0.0 0.0 ${height+0.105} rpy=0 0 0
- joint lidar_joint: origin xyz=0.22 0.0 ${height+0.125} rpy=0 0 -1.5708 -> xyz=0.22 0.0 ${height+0.125} rpy=0 0 0

Commit message: Arreglado problema del Range_finder

File: rover_description/src/description/rover.urdf (robot description, URDF)
Before this commit: robot sam_bot, 9 links, 8 joints
Links:
- removed link deph
- added link depth; visual box size=0.01 0.01 0.01
Joints:
- removed joint deph_joint
- added joint depth_joint: type fixed, parent base_link, child depth, origin xyz=0.405 0.0 ${height+0.095} rpy=0 0 0

Commit message: Arreglado completamente la pointcloud

File: rover_description/src/description/rover.urdf (robot description, URDF)
Before this commit: robot sam_bot, 8 links, 7 joints
Joints:
- joint depth_joint: origin xyz=0.405 0.0 ${height+0.095} rpy=0 0 0 -> xyz=0.405 0.0 ${height+0.095} rpy=-1.57079632679 0 -1.57079632679

Commit message: Implementacion rtabmap

File: rover_description/src/description/rover.urdf (robot description, URDF)
Before this commit: robot sam_bot, 8 links, 7 joints
Joints:
- joint camera_left_joint: origin xyz=0.405 0.06 ${height+0.095} rpy=0 0 0 -> xyz=0.405 0.06 ${height+0.095} rpy=-1.57079632679 0 -1.57079632679
- joint camera_right_joint: origin xyz=0.405 -0.06 ${height+0.095} rpy=0 0 0 -> xyz=0.405 -0.06 ${height+0.095} rpy=-1.57079632679 0 -1.57079632679
